File: KiCad_Project/Point Signal Box R2.kicad_sch (KiCad schematic)
At the start: 34 parts, among them J1 Alternate DCC, J2 SPDT on PM1, J3 SPDT on PM2, J4 As Needed, J5 Accessory Switch on Point Mot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, SW1 SW_SPDT, U1 TLP241B, U2 TLP241B, U3 TLP241B, U4 TLP241B

Commit message: Minor updates during editorial process
Parts:
- J2: value SPDT on PM1 -> To SPDT on PM1
- J3: value SPDT on PM2 -> To SPDT on PM2
Connections:
- net DCCJ: now also LED6.2 (Pin_2); no longer LED6.1 (Pin_1)
- net at J3.2 (Pin_2): now also LED6.1 (Pin_1); no longer LED6.2 (Pin_2)
Other:
- moved on the sheet: J2, J3, LED5, LED6
Changed lines of the file:
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@@
     )
   )
-  (global_label "DCCJ" (shape input) (at 181.61 96.52 0) (fields_autoplaced)
-    (effects (font (size 1.27 1.27)) (justify left))
-    (property "Intersheet References" "${INTERSHEET_REFS}" (id 0) (at 188.8007 96.4406 0)
-      (effects (font (size 1.27 1.27)) (justify left) hide)
+  (global_label "DCCJ" (shape input) (at 224.79 96.52 180) (fields_autoplaced)
+    (effects (font (size 1.27 1.27)) (justify right))
+    (property "Intersheet References" "${INTERSHEET_REFS}" (id 0) (at 217.5993 96.5994 0)
+      (effects (font (size 1.27 1.27)) (justify right) hide)
     )
   )
@@
     )
   )
-  (global_label "DCCJ" (shape input) (at 64.77 96.52 0) (fields_autoplaced)
-    (effects (font (size 1.27 1.27)) (justify left))
-    (property "Intersheet References" "${INTERSHEET_REFS}" (id 0) (at 71.9607 96.4406 0)
-      (effects (font (size 1.27 1.27)) (justify left) hide)
+  (global_label "DCCJ" (shape input) (at 109.22 96.52 180) (fields_autoplaced)
+    (effects (font (size 1.27 1.27)) (justify right))
+    (property "Intersheet References" "${INTERSHEET_REFS}" (id 0) (at 102.0293 96.4406 0)
+      (effects (font (size 1.27 1.27)) (justify right) hide)
     )
   )
@@
     (pin "2")
   )
-  (symbol (lib_id "Connector:Conn_01x03_Male") (at 195.58 107.95 90) (unit 1)
-    (in_bom yes) (on_board yes) (fields_autoplaced)
-    (property "Reference" "J3" (id 0) (at 195.58 110.49 90))
-    (property "Value" "SPDT on PM2" (id 1) (at 195.58 113.03 90))
-    (property "Footprint" "Connector_PinHeader_2.54mm:PinHeader_1x03_P2.54mm_Vertical" (id 2) (at 195.58 107.95 0)
-      (effects (font (size 1.27 1.27)) hide)
-    )
-    (property "Datasheet" "~" (id 3) (at 195.58 107.95 0)
+  (symbol (lib_id "Connector:Conn_01x03_Male") (at 167.64 99.06 0) (unit 1)
+    (in_bom yes) (on_board yes)
+    (property "Reference" "J3" (id 0) (at 165.1 99.06 90))
+    (property "Value" "To SPDT on PM2" (id 1) (at 171.45 104.14 0))
+    (property "Footprint" "Connector_PinHeader_2.54mm:PinHeader_1x03_P2.54mm_Vertical" (id 2) (at 167.64 99.06 0)
+      (effects (font (size 1.27 1.27)) hide)
+    )
+    (property "Datasheet" "~" (id 3) (at 167.64 99.06 0)
       (effects (font (size 1.27 1.27)) hide)
     )
@@
     (pin "3")
   )
-  (symbol (lib_id "Connector:Conn_01x03_Male") (at 78.74 107.95 90) (unit 1)
-    (in_bom yes) (on_board yes) (fields_autoplaced)
-    (property "Reference" "J2" (id 0) (at 78.74 110.49 90))
-    (property "Value" "SPDT on PM1" (id 1) (at 78.74 113.03 90))
-    (property "Footprint" "Connector_PinHeader_2.54mm:PinHeader_1x03_P2.54mm_Vertical" (id 2) (at 78.74 107.95 0)
-      (effects (font (size 1.27 1.27)) hide)
-    )
-    (property "Datasheet" "~" (id 3) (at 78.74 107.95 0)
+  (symbol (lib_id "Connector:Conn_01x03_Male") (at 60.96 99.06 0) (unit 1)
+    (in_bom yes) (on_board yes)
+    (property "Reference" "J2" (id 0) (at 58.42 99.06 90))
+    (property "Value" "To SPDT on PM1" (id 1) (at 60.96 104.14 0))
+    (property "Footprint" "Connector_PinHeader_2.54mm:PinHeader_1x03_P2.54mm_Vertical" (id 2) (at 60.96 99.06 0)
+      (effects (font (size 1.27 1.27)) hide)
+    )
+    (property "Datasheet" "~" (id 3) (at 60.96 99.06 0)
       (effects (font (size 1.27 1.27)) hide)
     )
@@
     (pin "2")
   )
-  (symbol (lib_id "Connector:Conn_01x02_Male") (at 168.91 96.52 0) (unit 1)
-    (in_bom yes) (on_board yes)
-    (property "Reference" "LED6" (id 0) (at 170.18 102.87 0))
-    (property "Value" "To Signal LED" (id 1) (at 160.02 96.52 0)
-      (effects (font (size 1.27 1.27)) hide)
-    )
-    (property "Footprint" "TerminalBlock_TE-Connectivity:TerminalBlock_TE_282834-2_1x02_P2.54mm_Horizontal" (id 2) (at 168.91 96.52 0)
-      (effects (font (size 1.27 1.27)) hide)
-    )
-    (property "Datasheet" "~" (id 3) (at 168.91 96.52 0)
+  (symbol (lib_id "Connector:Conn_01x02_Male") (at 233.68 99.06 180) (unit 1)
+    (in_bom yes) (on_board yes)
+    (property "Reference" "LED6" (id 0) (at 236.22 97.79 90))
+    (property "Value" "To Signal LED" (id 1) (at 242.57 99.06 0)
+      (effects (font (size 1.27 1.27)) hide)
+    )
+    (property "Footprint" "TerminalBlock_TE-Connectivity:TerminalBlock_TE_282834-2_1x02_P2.54mm_Horizontal" (id 2) (at 233.68 99.06 0)
+      (effects (font (size 1.27 1.27)) hide)
+    )
+    (property "Datasheet" "~" (id 3) (at 233.68 99.06 0)
       (effects (font (size 1.27 1.27)) hide)
     )
@@
     (pin "4")
   )
-  (symbol (lib_id "Connector:Conn_01x02_Male") (at 52.07 96.52 0) (unit 1)
-    (in_bom yes) (on_board yes)
-    (property "Reference" "LED5" (id 0) (at 53.34 102.87 0))
-    (property "Value" "To Signal LED" (id 1) (at 43.18 96.52 0))
-    (property "Footprint" "TerminalBlock_TE-Connectivity:TerminalBlock_TE_282834-2_1x02_P2.54mm_Horizontal" (id 2) (at 52.07 96.52 0)
-      (effects (font (size 1.27 1.27)) hide)
-    )
-    (property "Datasheet" "~" (id 3) (at 52.07 96.52 0)
+  (symbol (lib_id "Connector:Conn_01x02_Male") (at 114.3 96.52 0) (mirror y) (unit 1)
+    (in_bom yes) (on_board yes)
+    (property "Reference" "LED5" (id 0) (at 116.84 97.79 90))
+    (property "Value" "To Signal LED" (id 1) (at 111.76 104.14 0))
+    (property "Footprint" "TerminalBlock_TE-Connectivity:TerminalBlock_TE_282834-2_1x02_P2.54mm_Horizontal" (id 2) (at 114.3 96.52 0)
+      (effects (font (size 1.27 1.27)) hide)
+    )
+    (property "Datasheet" "~" (id 3) (at 114.3 96.52 0)
       (effects (font (size 1.27 1.27)) hide)
     )
@@
     )
     (path "/bcfee42a-a2a1-4347-aafa-48c497c5d3c6"
-      (reference "J2") (unit 1) (value "SPDT on PM1") (footprint "Connector_PinHeader_2.54mm:PinHeader_1x03_P2.54mm_Vertical")
+      (reference "J2") (unit 1) (value "To SPDT on PM1") (footprint "Connector_PinHeader_2.54mm:PinHeader_1x03_P2.54mm_Vertical")
     )
     (path "/16724819-e98d-4565-8e9e-29bb82faee74"
-      (reference "J3") (unit 1) (value "SPDT on PM2") (footprint "Connector_PinHeader_2.54mm:PinHeader_1x03_P2.54mm_Vertical")
+      (reference "J3") (unit 1) (value "To SPDT on PM2") (footprint "Connector_PinHeader_2.54mm:PinHeader_1x03_P2.54mm_Vertical")
     )
     (path "/04cf6992-2be1-4ba0-8ad4-843c5d37e550"
